File: hardware/picow_adapter/picow_adapter.kicad_sch (KiCad schematic)
At the start: 1 part

Commit message: update
Parts:
- added J1: Sensorclock, symbol Connector_Generic:Conn_02x10_Counter_Clockwise
- added Q1: DMG2305UX, Package_TO_SOT_SMD:SOT-23, symbol Simulation_SPICE:PMOS
Connections:
- net GND: now reaches A1.13 (GND), A1.18 (GND), A1.23 (GND), A1.28 (GND), A1.3 (GND), A1.38 (GND), A1.8 (GND)
- net GND: now also J1.10 (Pin_10), J1.17 (Pin_17), J1.18 (Pin_18), J1.19 (Pin_19), J1.20 (Pin_20), J1.8 (Pin_8)
- net at A1.39 (VSYS): now also Q1.2 (S)
- net at A1.40 (VBUS): now also Q1.1 (G)
- new net +5V: J1.2 (Pin_2), J1.4 (Pin_4), Q1.3 (D)
Other:
- moved on the sheet: A1

Commit message: update
Parts:
- added SW1: SW_Push, Button_Switch_SMD:SW_SPST_B3U-1000P, symbol Switch:SW_Push
- J1: footprint (none) -> Connector_PinSocket_2.54mm:PinSocket_2x10_P2.54mm_Vertical; symbol Connector_Generic:Conn_02x10_Counter_Clockwise -> Connector_Generic:Conn_02x10_Odd_Even
Connections:
- net GND: now also J1.6 (Pin_6), SW1.2
- net SPI0_SCK: now reaches A1.24 (GPIO18)
- net SPI0_SCK: now also J1.9 (Pin_9)
- net SPI0_TX: now reaches A1.25 (GPIO19)
- net SPI0_TX: now also J1.7 (Pin_7)
- net RESET: now reaches A1.30 (RUN)
- net RESET: now also SW1.1
- net I2C0_SDA: now reaches A1.6 (GPIO4)
- net I2C0_SDA: now also J1.3 (Pin_3)
- net I2C0_SCL: now reaches A1.7 (GPIO5)
- net I2C0_SCL: now also J1.5 (Pin_5)
- net ~{SHDN_3V3}: now reaches J1.1 (Pin_1)
- net HEATER_ENABLE: now reaches J1.11 (Pin_11)
- net TSL2561_INT: now reaches J1.12 (Pin_12)
- net DS3231_INT: now reaches J1.13 (Pin_13)
- net S1_S: now reaches J1.14 (Pin_14)
- net S1_A: now reaches J1.15 (Pin_15)
- net S1_B: now reaches J1.16 (Pin_16)

Commit message: update
Connections:
- net HEATER_ENABLE: now also A1.4 (GPIO2)
- net S1_A: now also A1.9 (GPIO6)
- net S1_B: now also A1.10 (GPIO7)
- net S1_S: now also A1.11 (GPIO8)
- net TSL2561_INT: now also A1.12 (GPIO9)
- net ~{SHDN_3V3}: now also A1.5 (GPIO3)
- net DS3231_INT: no longer names the net of J1.13 (Pin_13)
Changed lines of the file:
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@@
+    (stroke (width 0) (type default))
+  )
+  (wire (pts (xy 92.71 83.82) (xy 105.41 83.82))
     (stroke (width 0) (type default))
   )
@@
   )
   (wire (pts (xy 19.05 71.12) (xy 35.56 71.12))
+    (stroke (width 0) (type default))
+  )
+  (wire (pts (xy 92.71 66.04) (xy 105.41 66.04))
     (stroke (width 0) (type default))
   )
@@
     (stroke (width 0) (type default))
   )
+  (wire (pts (xy 92.71 81.28) (xy 105.41 81.28))
+    (stroke (width 0) (type default))
+  )
   (wire (pts (xy 118.11 109.22) (xy 118.11 113.03))
     (stroke (width 0) (type default))
@@
   )
   (wire (pts (xy 62.23 71.12) (xy 62.23 68.58))
-    (stroke (width 0) (type default))
-  )
-  (wire (pts (xy 19.05 86.36) (xy 35.56 86.36))
     (stroke (width 0) (type default))
   )
@@
     (stroke (width 0) (type default))
   )
+  (wire (pts (xy 92.71 78.74) (xy 105.41 78.74))
+    (stroke (width 0) (type default))
+  )
   (wire (pts (xy 62.23 93.98) (xy 62.23 99.06))
+    (stroke (width 0) (type default))
+  )
+  (wire (pts (xy 92.71 76.2) (xy 105.41 76.2))
     (stroke (width 0) (type default))
   )
@@
   )
   (wire (pts (xy 62.23 91.44) (xy 62.23 93.98))
+    (stroke (width 0) (type default))
+  )
+  (wire (pts (xy 92.71 63.5) (xy 105.41 63.5))
     (stroke (width 0) (type default))
   )
@@
     (effects (font (size 1.27 1.27)) (justify left bottom))
   )
+  (label "S1_S" (at 92.71 81.28 0) (fields_autoplaced)
+    (effects (font (size 1.27 1.27)) (justify left bottom))
+  )
   (label "I2C0_SDA" (at 92.71 68.58 0) (fields_autoplaced)
     (effects (font (size 1.27 1.27)) (justify left bottom))
   )
-  (label "DS3231_INT" (at 19.05 86.36 0) (fields_autoplaced)
+  (label "RESET" (at 143.51 63.5 0) (fields_autoplaced)
     (effects (font (size 1.27 1.27)) (justify left bottom))
   )
-  (label "RESET" (at 143.51 63.5 0) (fields_autoplaced)
+  (label "~{SHDN_3V3}" (at 92.71 66.04 0) (fields_autoplaced)
     (effects (font (size 1.27 1.27)) (justify left bottom))
   )
@@
     (effects (font (size 1.27 1.27)) (justify left bottom))
   )
+  (label "HEATER_ENABLE" (at 92.71 63.5 0) (fields_autoplaced)
+    (effects (font (size 1.27 1.27)) (justify left bottom))
+  )
   (label "SPI0_SCK" (at 143.51 96.52 0) (fields_autoplaced)
+    (effects (font (size 1.27 1.27)) (justify left bottom))
+  )
+  (label "S1_B" (at 92.71 78.74 0) (fields_autoplaced)
+    (effects (font (size 1.27 1.27)) (justify left bottom))
+  )
+  (label "S1_A" (at 92.71 76.2 0) (fields_autoplaced)
     (effects (font (size 1.27 1.27)) (justify left bottom))
   )
@@
     (effects (font (size 1.27 1.27)) (justify left bottom))
   )
+  (label "TSL2561_INT" (at 92.71 83.82 0) (fields_autoplaced)
+    (effects (font (size 1.27 1.27)) (justify left bottom))
+  )
